File: kicad/tractor_controller/tractor_controller.kicad_sch (KiCad schematic)
At the start: 3 parts, among them J1 Conn_01x04, J6 Conn_02x04_Odd_Even, U1 WeMos_mini

Commit message: final HW version
Parts:
- removed J1: Conn_01x04, symbol Connector_Generic:Conn_01x04
- added J2: Conn_01x05_Pin, symbol Connector:Conn_01x05_Pin
Connections:
- net +5V: now also J2.1 (Pin_1)
- net GND: now also J2.5 (Pin_5)
- net Pedal: now also J2.2 (Pin_2)
- net REVERSE: now reaches U1.13 (D6)
- net REVERSE: now also J2.4 (Pin_4)
- net Reverse renamed DRIVE
- net DRIVE: now also J2.3 (Pin_3)
